File: IDEHat.kicad_pcb (KiCad board)
At the start: 2 copper layers, 56 x 65 mm, 35 parts, among them J1 Pi, J2 IDE, U1 AT24CS32, U2 TXS0108EPW, U3 MCP23S17_SO, U4 MCP23S17_SO

Commit message: Initial commit
Parts:
- moved R4 141.7 mm to (90.0, 149.0), turned to 270 degrees
- moved ? 141.1 mm to (106.4, 180.7), turned to 0 degrees
- moved R7 138.7 mm to (86.2, 149.0), turned to 270 degrees
- moved R8 137.7 mm to (85.0, 149.0), turned to 270 degrees
- moved R10 136.4 mm to (82.4, 149.0), turned to 270 degrees
- moved R11 135.5 mm to (81.2, 149.0), turned to 270 degrees
- moved R6 135.5 mm to (87.5, 149.0), turned to 270 degrees
- moved R9 133.8 mm to (83.7, 149.0), turned to 270 degrees
- moved R5 132.5 mm to (88.8, 149.0), turned to 270 degrees
- moved D1 130.0 mm to (106.5, 163.0), turned to 0 degrees
- moved D3 128.9 mm to (90.4, 145.5)
- moved D9 128.6 mm to (78.5, 145.5)
- moved D5 126.5 mm to (86.5, 145.5)
- moved R3 125.4 mm to (103.0, 163.0), turned to 180 degrees
- moved D6 125.0 mm to (84.6, 145.5)
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Routing:
- net +5V: track 210.8 -> 195.7 mm
- net Net-(D9-Pad1): track 0.00 -> 3.56 mm
- net Net-(D2-Pad1): track 0.00 -> 3.31 mm
- net Net-(D8-Pad1): track 0.00 -> 2.95 mm
- net Net-(D3-Pad1): track 0.00 -> 2.84 mm
- net Net-(D7-Pad1): track 0.00 -> 2.63 mm
- net Net-(D4-Pad1): track 0.00 -> 2.52 mm
- net Net-(D6-Pad1): track 0.00 -> 2.31 mm
- net Net-(D5-Pad1): track 0.00 -> 2.26 mm
- net GND: track 26.4 -> 28.6 mm
- net Net-(R9-Pad2): track 0.00 -> 1.94 mm
- net Net-(R8-Pad2): track 0.00 -> 1.94 mm
- net Net-(R5-Pad2): track 0.00 -> 1.94 mm
- net Net-(R7-Pad2): track 0.00 -> 1.94 mm
- net Net-(R6-Pad2): track 0.00 -> 1.94 mm
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Other:
- board size 56 x 65 mm -> 65 x 56 mm
- board text added: "ATA/ATAPI Hat Rev. A Tobias Mädel 2020"
- board text added: "JLCJLCJLCJLC"
- board text added: "tbspace.de"
