File: ATAPIHat.kicad_pcb (KiCad board)
At the start: 2 copper layers, 65 x 56 mm, 35 parts, among them J1 Pi, J2 IDE, U1 AT24CS32, U2 TXS0108EPW, U3 MCP23S17_SO, U4 MCP23S17_SO

Commit message: ATAPIHat Rev A Errata
Connections:
- net /3V_CS renamed /3V_CE1
- J1 pad 24: Net-(J1-Pad24) -> /3V_CE0
- U2 pad 15: Net-(U2-Pad15) -> /CE0
- U2 pad 20: /CS -> /CE1
- U2 pad 6: Net-(U2-Pad6) -> /3V_CE0
- U3 pad 11: /CS -> /CE1
- U3 pad 18: GND -> +5V
- U4 pad 11: /CS -> /CE0
- U4 pad 18: GND -> +5V
Routing:
- net /CS: track 47.0 -> 0.00 mm, vias 2 -> 0
- net /CE0: track 0.00 -> 42.4 mm, vias 0 -> 4
- net /3V_CE0: track 0.00 -> 21.3 mm
- net /CE1: track 0.00 -> 16.4 mm
- net +5V: track 195.7 -> 202.0 mm
- net /MISO: track 52.1 -> 53.3 mm
Other:
- board text added: "ATA/ATAPI Hat Rev. B Tobias Mädel 2020"
- board text removed: "ATA/ATAPI Hat Rev. A Tobias Mädel 2020"
